File: HW/REV2/KicadV2/xyp-gpib.kicad_pcb (KiCad board)
At the start: 2 copper layers, 54 x 15 mm, 25 parts, among them J1 USB_C_Receptacle_USB2.0, SW1 SW_Push, U1 ATmega32U4-MU, Y1 CX2016DB16000D0WZRC1

Commit message: GPIBee is available
- GPIBee availability / link sharing
- Adding more "proven to work"devices.
- Some BOM adjustments (was raised as Issue and this addresses it)
- Share a beautifully done project: Zandan Khan's XyphroLabs-USBGpib-DMM4050
Parts:
- C5, C6: value 8pF -> 18pF
- R7: value 10k -> 5k1
